File: SAM3S_SPARTAN6/i.MX283_Board.kicad_pcb (KiCad board)
At the start: 4 copper layers, 95 parts, among them U11 ZLDO1117G33TA, X401 12MHz

Commit message: Routing
Parts:
- added DP3: DIODE, opendous:SM0603_Opendous, F.Cu at (31.5, 115.5)
- added JMS2: USB-MINI, Connect:USB_Mini-B, F.Cu at (24.0, 118.2)
- added RUF1: 27, SM0603, F.Cu at (31.6, 117.2)
- added RUF2: 27, SM0603, F.Cu at (31.7, 118.7)
- added XF2: 6MHz, resonator:CSTCR6M00G53Z, F.Cu at (67.9, 129.1)
- CF39, RF18, RF19, RF20: moved to B.Cu
- moved CF40 86.9 mm to (64.4, 129.8), turned to 90 degrees
- moved CF38 85.9 mm to (71.3, 127.3), turned to 270 degrees
- moved CF37 85.6 mm to (61.6, 128.5), turned to 90 degrees
- moved CF41 84.4 mm to (71.3, 129.8), turned to 90 degrees
- moved LF11 83.1 mm to (57.9, 130.9)
- moved CF36 82.9 mm to (57.7, 128.6)
- moved DP1 80.3 mm to (78.8, 123.6), turned to 180 degrees
- moved RF17 77.4 mm to (74.2, 121.9), turned to 180 degrees
- moved RF15 77.1 mm to (78.6, 119.6), turned to 180 degrees
- moved CF39 77.0 mm to (68.2, 121.3), turned to 180 degrees
- moved RF16 76.8 mm to (74.2, 123.4)
- moved RF21 76.3 mm to (58.9, 125.8), turned to 90 degrees
- moved RF14 75.5 mm to (78.6, 121.1), turned to 180 degrees
- moved RF18 75.3 mm to (68.0, 123.3), turned to 180 degrees
- moved C74 75.1 mm to (46.9, 127.5)
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Connections:
- US1 pad 88: (no net) -> Net-(RUF1-Pad2)
- US1 pad 89: (no net) -> Net-(RUF2-Pad2)
Routing:
- net /spartan6/F_TMS: track 0.00 -> 85.9 mm, vias 0 -> 3
- net /spartan6/F_TCK: track 0.13 -> 85.1 mm, vias 0 -> 4
- net /SAM3M/JTDI: track 0.00 -> 82.0 mm, vias 0 -> 2
- net /spartan6/F_TDI: track 0.00 -> 66.0 mm, vias 0 -> 3
- net /spartan6/F_TDO: track 0.00 -> 38.5 mm, vias 0 -> 1
- net +3.3VDAC: track 100.0 -> 76.4 mm, vias 29 -> 23
- net +3.3V: track 0.00 -> 18.9 mm, vias 0 -> 1
- net +5VA: track 0.00 -> 18.1 mm, vias 0 -> 1
- net Net-(FT1-Pad7): track 0.00 -> 11.9 mm
- net VDD5V: track 24.3 -> 16.0 mm
- net Net-(CF40-Pad2): track 0.00 -> 6.45 mm
- net Net-(FT1-Pad8): track 0.00 -> 6.45 mm
- net Net-(CF41-Pad2): track 0.00 -> 6.22 mm
- net Net-(CF38-Pad1): track 0.00 -> 5.53 mm, vias 0 -> 1
- net Net-(FT1-Pad2): track 0.00 -> 5.36 mm
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- added copper zone on B.Cu, net GND
- added copper zone on F.Cu, net GND
Other:
- board text removed: "F_TDO"
- board text removed: "P_TDI"
- board text removed: "TDO"

Commit message: Routing almost finished
Parts:
- C76, RF21: moved to B.Cu
- moved C76 17.4 mm to (30.2, 112.6), turned to 270 degrees
- moved CF22 13.0 mm to (61.0, 109.3), turned to 270 degrees
- moved RF21 7.16 mm to (65.4, 122.9), turned to 0 degrees
- moved C74 6.82 mm to (53.4, 129.4), turned to 90 degrees
- moved CF35 6.15 mm to (48.0, 116.0)
- moved CF30 3.13 mm to (49.0, 109.1)
- moved CF26 2.14 mm to (68.9, 110.0)
- moved CF32 1.65 mm to (69.8, 110.7)
Routing:
- net +3.3VDAC: track 76.4 -> 201.3 mm, vias 23 -> 22
- net VDD5V: track 16.0 -> 130.2 mm, vias 2 -> 3
- net +3.3VP: track 36.2 -> 107.5 mm
- net /serial_interface/RXD: track 0.00 -> 54.3 mm, vias 0 -> 4
- net /SAM3M/SAM_RX: track 0.00 -> 52.1 mm, vias 0 -> 4
- net /SAM3M/SNRD: track 0.00 -> 50.2 mm, vias 0 -> 4
- net /SAM3M/SNWE: track 0.00 -> 43.2 mm, vias 0 -> 4
- net /spartan6/F_TDI: track 66.0 -> 108.6 mm, vias 3 -> 6
- net /SAM3M/AD4: track 36.1 -> 0.00 mm, vias 1 -> 0
- net Net-(RUF2-Pad2): track 0.00 -> 24.4 mm, vias 0 -> 2
- net Net-(RUF1-Pad2): track 0.00 -> 22.4 mm, vias 0 -> 2
- net GND: track 12.7 -> 20.8 mm, vias 7 -> 11
- net +5VA: track 18.1 -> 24.4 mm
- net Net-(DP1-Pad1): track 0.00 -> 4.59 mm
- net Net-(DP3-Pad1): track 0.00 -> 3.71 mm
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
Commit message: Finishing routing, adding gerber files
Parts:
- added TH1: CONN_1, opendous:1Pin_12mil_VIA, F.Cu at (21.3, 137.9)
- added TH10: CONN_1, opendous:1Pin_12mil_VIA, F.Cu at (31.5, 137.9)
- added TH11: CONN_1, opendous:1Pin_12mil_VIA, F.Cu at (69.6, 137.9)
- added TH12: CONN_1, opendous:1Pin_12mil_VIA, F.Cu at (23.9, 137.9)
- added TH13: CONN_1, opendous:1Pin_12mil_VIA, F.Cu at (54.3, 137.9)
- added TH14: CONN_1, opendous:1Pin_12mil_VIA, F.Cu at (51.8, 137.9)
- added TH15: CONN_1, opendous:1Pin_12mil_VIA, F.Cu at (26.4, 137.9)
- added TH16: CONN_1, opendous:1Pin_12mil_VIA, F.Cu at (59.4, 137.9)
- added TH17: CONN_1, opendous:1Pin_12mil_VIA, F.Cu at (44.2, 137.9)
- added TH18: CONN_1, opendous:1Pin_12mil_VIA, F.Cu at (41.6, 137.9)
- added TH19: CONN_1, opendous:1Pin_12mil_VIA, F.Cu at (39.1, 137.9)
- added TH2: CONN_1, opendous:1Pin_12mil_VIA, F.Cu at (46.7, 137.9)
- added TH20: CONN_1, opendous:1Pin_12mil_VIA, F.Cu at (49.3, 137.9)
- added TH21: CONN_1, opendous:1Pin_12mil_VIA, F.Cu at (21.9, 67.4)
- added TH22: CONN_1, opendous:1Pin_12mil_VIA, F.Cu at (27.0, 67.4)
- added TH23: CONN_1, opendous:1Pin_12mil_VIA, F.Cu at (44.8, 67.4)
- added TH24: CONN_1, opendous:1Pin_12mil_VIA, F.Cu at (29.6, 67.4)
- added TH25: CONN_1, opendous:1Pin_12mil_VIA, F.Cu at (42.3, 67.4)
- added TH26: CONN_1, opendous:1Pin_12mil_VIA, F.Cu at (47.4, 67.4)
- added TH27: CONN_1, opendous:1Pin_12mil_VIA, F.Cu at (32.1, 67.4)
- added TH28: CONN_1, opendous:1Pin_12mil_VIA, F.Cu at (49.9, 67.4)
- added TH29: CONN_1, opendous:1Pin_12mil_VIA, F.Cu at (34.6, 67.4)
- added TH3: CONN_1, opendous:1Pin_12mil_VIA, F.Cu at (36.6, 137.9)
- added TH30: CONN_1, opendous:1Pin_12mil_VIA, F.Cu at (39.7, 67.4)
- added TH31: CONN_1, opendous:1Pin_12mil_VIA, F.Cu at (21.3, 125.2)
- added TH32: CONN_1, opendous:1Pin_12mil_VIA, F.Cu at (21.3, 130.3)
- added TH33: CONN_1, opendous:1Pin_12mil_VIA, F.Cu at (72.1, 137.9)
- added TH34: CONN_1, opendous:1Pin_12mil_VIA, F.Cu at (74.7, 137.9)
- added TH35: CONN_1, opendous:1Pin_12mil_VIA, F.Cu at (21.3, 135.3)
- added TH36: CONN_1, opendous:1Pin_12mil_VIA, F.Cu at (21.3, 132.8)
- added TH37: CONN_1, opendous:1Pin_12mil_VIA, F.Cu at (21.3, 127.7)
- added TH38: CONN_1, opendous:1Pin_12mil_VIA, F.Cu at (37.2, 67.4)
- added TH39: CONN_1, opendous:1Pin_12mil_VIA, F.Cu at (24.5, 67.4)
- added TH4: CONN_1, opendous:1Pin_12mil_VIA, F.Cu at (56.9, 137.9)
- added TH40: CONN_1, opendous:1Pin_12mil_VIA, F.Cu at (52.4, 67.4)
- added TH41: CONN_1, opendous:1Pin_12mil_VIA, F.Cu at (55.0, 67.4)
- added TH42: CONN_1, opendous:1Pin_12mil_VIA, F.Cu at (57.5, 67.4)
- added TH43: CONN_1, opendous:1Pin_12mil_VIA, F.Cu at (60.0, 67.4)
- added TH44: CONN_1, opendous:1Pin_12mil_VIA, F.Cu at (65.1, 67.4)
- added TH45: CONN_1, opendous:1Pin_12mil_VIA, F.Cu at (62.6, 67.4)
- added TH46: CONN_1, opendous:1Pin_12mil_VIA, F.Cu at (67.7, 67.4)
- added TH47: CONN_1, opendous:1Pin_12mil_VIA, F.Cu at (70.2, 67.4)
- added TH48: CONN_1, opendous:1Pin_12mil_VIA, F.Cu at (75.3, 67.4)
- added TH49: CONN_1, opendous:1Pin_12mil_VIA, F.Cu at (72.8, 67.4)
- added TH5: CONN_1, opendous:1Pin_12mil_VIA, F.Cu at (62.0, 137.9)
- added TH50: CONN_1, opendous:1Pin_12mil_VIA, F.Cu at (77.8, 67.4)
- added TH6: CONN_1, opendous:1Pin_12mil_VIA, F.Cu at (28.9, 137.9)
- added TH7: CONN_1, opendous:1Pin_12mil_VIA, F.Cu at (34.0, 137.9)
- added TH8: CONN_1, opendous:1Pin_12mil_VIA, F.Cu at (64.5, 137.9)
- added TH9: CONN_1, opendous:1Pin_12mil_VIA, F.Cu at (67.0, 137.9)
Connections:
- PSA1 pad 24: +3.3VP -> GND
- PSA1 pad 27: /SAM3M/AD4 -> +3.3VP
- UF1 pad 1: (no net) -> /SAM3M/AS10
- US1 pad 3: /SAM3M/AD4 -> (no net)
- US1 pad 54: (no net) -> /SAM3M/AS10
Routing:
- net /SAM3M/JNRST: track 0.00 -> 66.3 mm, vias 0 -> 6
- net /SAM3M/AS10: track 0.00 -> 30.5 mm, vias 0 -> 2
- net +3.3VP: track 107.5 -> 112.5 mm
- net /spartan6/F_TDI: track 108.6 -> 108.5 mm, vias 6 -> 5
