File: SAM3S_SPARTAN6/i.MX283_Board.kicad_pcb (KiCad board)
At the start: 4 copper layers, 150 parts, among them U11 ZLDO1117G33TA, X401 12MHz

Commit message: Added files via upload
Parts:
- removed C396, C397, C398, C399, C400: 0.1uF, SM0603
- removed C74, C76: 33uF, SM1206
- removed C75: 100n, SM0603
- removed D8, D9: LED, SM0603
- removed DP3: DIODE, opendous:SM0603_Opendous
- removed JMS2: USB-MINI, Connect:USB_Mini-B
- removed PSA1: CONN_02X14, Socket_Strips:Socket_Strip_Straight_2x14
- removed R33: 1k, SM0603
- removed RUF1, RUF2: 27, SM0603
- removed TH1, TH10, TH11, TH12, TH13, TH14, TH15, TH16, TH17, TH18, TH19, TH2, TH20, TH21, TH22, TH23, TH24, TH25, TH26, TH27, TH28, TH29, TH3, TH30, TH31, TH32, TH33, TH34, TH35, TH36, TH37, TH38, TH39, TH4, TH40, TH41, TH42, TH43, TH44, TH45, TH46, TH47, TH48, TH49, TH5, TH50, TH6, TH7, TH8, TH9: CONN_1, opendous:1Pin_12mil_VIA
- removed U11: ZLDO1117G33TA, LT1117
- removed US1: ATSAM3S2CA-AU, Housings_QFP:LQFP-100_14x14mm_Pitch0.5mm
- removed X401: 12MHz, ABM8G
- added C1: 4.7uF, opendous:SM1206_Opendous, F.Cu at (106.5, 87.7)
- added C2: 33uF, opendous:SM1206_Opendous, F.Cu at (114.1, 97.5)
- added C3: 100nF, opendous:SM0603, F.Cu at (116.2, 95.3)
- added C4: 33uF, opendous:SM1206_Opendous, F.Cu at (106.0, 98.0)
- added C413: 0.1uF, opendous:SM0603, F.Cu at (94.8, 135.5)
- added C414: 0.1uF, opendous:SM0603, F.Cu at (70.3, 132.6)
- added C415: 4.7uF, opendous:SM1206_Opendous, F.Cu at (81.2, 141.1)
- added C416: 0.1uF, opendous:SM0603, F.Cu at (97.7, 115.6)
- added C417: 1uF, opendous:SM0603, F.Cu at (82.7, 135.6)
- added C418: 1uF, opendous:SM0603, F.Cu at (103.2, 114.3)
- added C419: 1uF, opendous:SM0603, F.Cu at (103.2, 116.2)
- added C420: 0.1uF, opendous:SM0603, F.Cu at (97.7, 114.1)
- added C421: 0.1uF, opendous:SM0603, F.Cu at (117.4, 105.4)
- added C422: 0.1uF, opendous:SM0603, F.Cu at (81.1, 135.5)
- added C423: 0.1uF, opendous:SM0603, F.Cu at (86.1, 135.5)
- added C424: 0.1uF, opendous:SM0603, F.Cu at (97.9, 117.1)
- added C425: 2.2uF, opendous:SM0603, F.Cu at (70.8, 131.0)
- added C426: 2.2uF, opendous:SM0603, F.Cu at (74.6, 109.2)
- added CXOUT1: 6.8pF, opendous:SM0603, F.Cu at (102.2, 128.7)
- added CXOUT2: 6.8pF, opendous:SM0603, F.Cu at (102.2, 126.2)
- added CXST1: 22pF, opendous:SM0603, F.Cu at (103.4, 119.2)
- added CXST2: 22pF, opendous:SM0603, F.Cu at (103.4, 120.9)
- added J1: CONN_3X1F, CONAL:pin_array_1x3, F.Cu at (113.4, 121.5)
- added J401: USB-MINI, CONAL:m-pad-2.1-USB-MINI-B, F.Cu at (63.0, 152.3)
- added JP401: JUMPER, CONAL:pin_array_1x2, F.Cu at (98.3, 104.2)
- added JP402: JUMPER, CONAL:pin_array_1x2, F.Cu at (93.4, 139.6)
- added L401: 2A 120 ohm, opendous:SM0805, F.Cu at (99.3, 111.7)
- added L402: 2A 120 ohm, opendous:SM0805, F.Cu at (100.7, 115.2)
- added LED1: LED, opendous:SM0603, F.Cu at (90.0, 108.0)
- added LED2: LED, opendous:SM0603, F.Cu at (107.1, 92.8)
- added P1: CONN_13X2, CONN_02X13:pin_array_13x2, F.Cu at (58.3, 123.6)
- added P2: CONN_8X2, CONAL:pin_array_8x2, F.Cu at (84.3, 153.9)
- added R1: 0, opendous:SM0603, F.Cu at (106.1, 109.7)
- added R2: 0, opendous:SM0603, F.Cu at (65.0, 144.5)
- added R3: 22, opendous:SM0603, F.Cu at (63.4, 144.5)
- added R4: 22, opendous:SM0603, F.Cu at (61.9, 144.5)
- added R401: 10K, opendous:SM0603, F.Cu at (108.0, 123.4)
- added R402: 10K, opendous:SM0603, F.Cu at (87.1, 108.9)
- added R403: 10k, opendous:SM0603, F.Cu at (91.8, 106.1)
- added R404: 10K, opendous:SM0603, F.Cu at (86.6, 139.9)
- added R6: 470, opendous:SM0603, F.Cu at (105.5, 92.8)
- added R7: 10K, opendous:SM0603, F.Cu at (111.4, 95.4)
- added R8: 0, opendous:SM0603, F.Cu at (107.8, 109.5)
- added SW401: SW_PUSH, discret:SW_PUSH_SMALL, F.Cu at (112.7, 113.9)
- added U1: STMPS2141STR, sot:SOT23-5, F.Cu at (110.9, 91.0)
- added U1401: STM32F4_LQFP144, Housings_QFP:LQFP-144_20x20mm_Pitch0.5mm, F.Cu at (83.9, 122.4)
- added U2: ZLDO1117G33TA, sot:SOT223, F.Cu at (111.2, 104.6)
- added XOUT401: 32.768kHz, resonator:XC32.778KhZ, F.Cu at (99.4, 127.5)
- added XST1: 12MHz, ABM8G:ABM8G, F.Cu at (98.7, 120.9)
- C401: value 0.1uF -> 1uF; footprint SM0603 -> opendous:SM0603; moved to F.Cu
- C402, C403: value 20pF -> 0.1uF; footprint SM0603 -> opendous:SM0603; moved to F.Cu
- C404, C405, C408, C409, C410, CF1, CF10, CF11, CF12, CF13, CF14, CF16, CF17, CF18, CF19, CF2, CF20, CF21, CF23, CF24, CF25, CF26, CF27, CF28, CF3, CF31, CF33, CF4, CF5, CF6, CF7, CF8, CF9, RF1, RF2, RF3, RF4, RF6, RF7: footprint SM0603 -> opendous:SM0603; moved to F.Cu
- C406, C411: value 1uF -> 0.1uF; footprint SM0603 -> opendous:SM0603; moved to F.Cu
- C407: value 4.7uF -> 0.1uF; footprint SM1206 -> opendous:SM0603
- C412: value 4.7uF -> 0.1uF; footprint SM1206 -> opendous:SM0603; moved to F.Cu
- CF15, CF22, CF29, CF30, CF34, CF35: footprint SM1206_Opendous -> opendous:SM1206_Opendous; moved to F.Cu
- CF32: footprint SM1206_Opendous -> opendous:SM1206_Opendous
- CF39, RF18, RF19, RF20, RF21: moved to F.Cu
- DF1, RF5: footprint SM0603 -> opendous:SM0603
- JMS1: footprint Connect:USB_Mini-B -> CONAL:m-pad-2.1-USB-MINI-B
- PFIO1: footprint Socket_Strips:Socket_Strip_Straight_2x18 -> CONN_18X2:pin_array_18x2
- PFIO2: footprint Socket_Strips:Socket_Strip_Straight_2x12 -> CONN_02X14:pin_array_13x2
- PS1: footprint Connect:JACK_ALIM -> J5:J5
- R5: value 1k -> 47K; footprint SM0603 -> opendous:SM0603
- UF2, UF3: footprint SMD_Packages:SOT-223 -> sot:SOT223
- moved PS1 90.4 mm to (119.0, 50.5), turned to 270 degrees
- moved CF35 85.5 mm to (112.7, 60.0), turned to 180 degrees
- moved C405 82.8 mm to (114.4, 93.0)
- moved UF3 75.8 mm to (111.2, 65.3), turned to 180 degrees
- moved CF30 73.5 mm to (112.6, 72.1)
- moved C401 71.8 mm to (93.2, 135.5)
- moved C410 69.9 mm to (97.0, 129.6), turned to 270 degrees
- moved R5 69.4 mm to (108.7, 94.4), turned to 90 degrees
- moved CF11 67.4 mm to (116.6, 64.5), turned to 90 degrees
- moved C402 66.6 mm to (108.1, 120.5), turned to 270 degrees
- moved C404 65.6 mm to (91.6, 109.3), turned to 90 degrees
- moved C409 61.7 mm to (96.5, 122.2), turned to 90 degrees
- moved CF4 59.6 mm to (116.9, 76.2)
- moved UF2 59.1 mm to (111.1, 77.8), turned to 180 degrees
- moved C406 58.5 mm to (91.7, 135.5)
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Connections:
- C401 pad 1: +3.3VP -> 3V3
- C402 pad 1: Net-(C402-Pad1) -> /STM32F4/NRST
- C403 pad 1: Net-(C403-Pad1) -> 3V3
- C404 pad 1: +3.3VP -> 3V3
- C405 pad 1: +3.3VP -> 3V3
- C406 pad 1: +3.3VP -> 3V3
- C407 pad 1: +3.3VP -> 3V3
- C408 pad 1: +1.8V -> 3V3
- C409 pad 1: +1.8V -> 3V3
- C410 pad 1: +1.8V -> 3V3
- C411 pad 1: +1.8V -> 3V3
- C412 pad 1: +1.8V -> 3V3
- CF35 pad 1: VDD5V -> +5V
- CF36 pad 1: VDD5V -> +5V
- DF1 pad 1: /spartan6/IO7 -> /spartan6/IO16
- FT1 pad 1: (no net) -> Net-(FT1-Pad1)
- FT1 pad 11: (no net) -> Net-(FT1-Pad11)
- FT1 pad 12: (no net) -> Net-(FT1-Pad12)
- FT1 pad 13: (no net) -> Net-(FT1-Pad13)
- FT1 pad 15: (no net) -> Net-(FT1-Pad15)
- FT1 pad 16: (no net) -> Net-(FT1-Pad16)
- FT1 pad 17: (no net) -> /serial_interface/nSRST
- FT1 pad 19: (no net) -> Net-(FT1-Pad19)
- FT1 pad 20: /SAM3M/JNRST -> /STM32F4/NJTRST
- FT1 pad 23: /SAM3M/JTDI -> /STM32F4/JTDI
- FT1 pad 27: (no net) -> Net-(FT1-Pad27)
- FT1 pad 28: (no net) -> Net-(FT1-Pad28)
- FT1 pad 29: (no net) -> Net-(FT1-Pad29)
- FT1 pad 30: (no net) -> Net-(FT1-Pad30)
- FT1 pad 32: (no net) -> Net-(FT1-Pad32)
- FT1 pad 33: (no net) -> Net-(FT1-Pad33)
- FT1 pad 35: (no net) -> Net-(FT1-Pad35)
- FT1 pad 36: (no net) -> Net-(FT1-Pad36)
- FT1 pad 37: (no net) -> Net-(FT1-Pad37)
- FT1 pad 38: (no net) -> Net-(FT1-Pad38)
- FT1 pad 40: /SAM3M/SAM_RX -> /serial_interface/TXD
- FT1 pad 41: (no net) -> Net-(FT1-Pad41)
- FT1 pad 48: (no net) -> Net-(FT1-Pad48)
- JMS1 pad 4: (no net) -> Net-(JMS1-Pad4)
- LF11 pad 1: VDD5V -> +5V
- PFIO1 pad 19: (no net) -> GND
- PFIO2 pad 1: /spartan6/IO54 -> /spartan6/IO55
- PFIO2 pad 10: /spartan6/IO47 -> /spartan6/IO46
- PFIO2 pad 11: /spartan6/IO44 -> /spartan6/IO45
- PFIO2 pad 12: /spartan6/IO45 -> /spartan6/IO44
- PFIO2 pad 13: /spartan6/IO42 -> /spartan6/IO43
- PFIO2 pad 14: /spartan6/IO43 -> /spartan6/IO42
- PFIO2 pad 2: /spartan6/IO55 -> /spartan6/IO54
- PFIO2 pad 3: /spartan6/IO52 -> /spartan6/IO53
- PFIO2 pad 4: /spartan6/IO53 -> /spartan6/IO52
- PFIO2 pad 5: /spartan6/IO50 -> /spartan6/IO51
- PFIO2 pad 6: /spartan6/IO51 -> /spartan6/IO50
- PFIO2 pad 7: /spartan6/IO48 -> /spartan6/IO49
- PFIO2 pad 8: /spartan6/IO49 -> /spartan6/IO48
- PFIO2 pad 9: /spartan6/IO46 -> /spartan6/IO47
- PS1 pad 1: VDD5V -> VDD4P2
- PS1 pad 3: (no net) -> Net-(PS1-Pad3)
- R5 pad 1: GND -> 3V3
- UF1 pad 1: /SAM3M/AS10 -> /STM32F4/AS11
- UF1 pad 10: (no net) -> /STM32F4/DS0
- UF1 pad 11: /SAM3M/SNWAIT -> /STM32F4/AS7
- UF1 pad 12: /spartan6/IO7 -> /STM32F4/AS6
- UF1 pad 137: /SAM3M/DS1 -> /spartan6/IO5
- UF1 pad 138: /SAM3M/DS2 -> /STM32F4/DS2
- UF1 pad 139: /SAM3M/DS3 -> /STM32F4/DS3
- UF1 pad 14: (no net) -> /STM32F4/NOE
- UF1 pad 140: /SAM3M/DS4 -> /STM32F4/DS7
- UF1 pad 141: /SAM3M/DS5 -> /STM32F4/DS6
- UF1 pad 142: /SAM3M/DS6 -> /STM32F4/DS5
- UF1 pad 143: /SAM3M/DS7 -> /STM32F4/DS4
- UF1 pad 15: /SAM3M/SNWE -> /STM32F4/NWE
- UF1 pad 16: /SAM3M/AS9 -> /STM32F4/NWAIT
- UF1 pad 17: /SAM3M/CLK_F -> /spartan6/CLK_FPGA
- UF1 pad 2: (no net) -> /STM32F4/AS10
- UF1 pad 21: /SAM3M/AS8 -> /spartan6/IO4
- UF1 pad 22: (no net) -> /spartan6/IO10
- UF1 pad 23: /SAM3M/SNRD -> /spartan6/IO3
- UF1 pad 24: /SAM3M/AS13 -> /STM32F4/CS
- UF1 pad 26: (no net) -> /spartan6/IO11
- UF1 pad 27: /SAM3M/AS12 -> /spartan6/IO7
- UF1 pad 29: /SAM3M/AS11 -> /spartan6/IO2
- UF1 pad 30: (no net) -> /spartan6/IO12
- UF1 pad 32: (no net) -> /spartan6/IO13
- UF1 pad 33: (no net) -> /spartan6/IO14
- UF1 pad 34: (no net) -> /STM32F4/NBL0
- UF1 pad 35: (no net) -> /STM32F4/NBL1
- UF1 pad 39: /SAM3M/AS7 -> /spartan6/IO16
- UF1 pad 40: /SAM3M/AS6 -> /spartan6/IO15
- UF1 pad 41: /SAM3M/AS5 -> /STM32F4/AS5
- UF1 pad 43: /SAM3M/AS4 -> /STM32F4/AS4
- UF1 pad 44: /SAM3M/AS3 -> /STM32F4/AS3
- UF1 pad 45: /SAM3M/AS2 -> /STM32F4/AS2
- UF1 pad 46: /SAM3M/AS1 -> /STM32F4/AS1
- UF1 pad 47: /SAM3M/AS0 -> /STM32F4/AS0
- UF1 pad 5: (no net) -> /STM32F4/AS9
- UF1 pad 6: (no net) -> /STM32F4/AS8
- UF1 pad 7: /SAM3M/DS0 -> /STM32F4/AS13
- UF1 pad 71: (no net) -> Net-(UF1-Pad71)
- UF1 pad 72: (no net) -> Net-(UF1-Pad72)
- UF1 pad 73: (no net) -> Net-(UF1-Pad73)
- UF1 pad 8: (no net) -> /STM32F4/AS12
- UF1 pad 9: /SAM3M/SNCS -> /STM32F4/DS1
- UF3 pad 3: VDD5V -> +5V
Routing:
- net 3V3: track 0.00 -> 255.3 mm, vias 0 -> 15
- net /STM32F4/VBUS: track 0.00 -> 131.5 mm, vias 0 -> 2
- net +3.3VP: track 112.5 -> 0.00 mm, vias 10 -> 0
- net +5V: track 0.00 -> 100.3 mm, vias 0 -> 1
- net VDD4P2: track 0.00 -> 87.5 mm
- net VDD5V: track 130.2 -> 44.4 mm, vias 3 -> 2
- net /SAM3M/JTDI: track 82.4 -> 0.00 mm, vias 4 -> 0
- net /spartan6/F_TDO: track 38.5 -> 114.1 mm, vias 1 -> 4
- net /SAM3M/JNRST: track 66.3 -> 0.00 mm, vias 6 -> 0
- net +1.8V: track 66.0 -> 0.00 mm, vias 8 -> 0
- net +3.3VDAC: track 201.3 -> 263.8 mm, vias 22 -> 15
- net /STM32F4/AS0: track 0.00 -> 58.6 mm
- net /STM32F4/AS1: track 0.00 -> 57.2 mm
- net /STM32F4/AS2: track 0.00 -> 55.8 mm
- net /STM32F4/AS3: track 0.00 -> 54.4 mm
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Other:
- board outline added: 72.4 x 109.9 mm
- copper layers 4 -> 2
- net class DDR2 removed
- net class Default: clearance 0.099 -> 0.2; trace_width 0.1 -> 0.25; via_dia 0.4 -> 0.6; via_drill 0.2032 -> 0.4
- net class iNAND removed
- rule trace_clearance: 0.099 -> 0.2
- rule trace_min: 0.09 -> 0.15
- board text removed: "1"
- board text removed: "2"
- board text removed: "A"
- board text removed: "K"

Commit message: Added files via upload
Parts:
- moved C404 0.94 mm to (92.4, 109.7), turned to 0 degrees
- moved CF1 0.62 mm to (90.7, 69.3)
- moved C403 0.59 mm to (70.1, 118.5)
- moved C421 0.47 mm to (116.9, 105.4)
- moved R402 0.44 mm to (87.5, 109.0)
- moved C411 0.41 mm to (85.5, 108.9)
- moved C409 0.38 mm to (96.5, 121.8)
- moved C414 0.37 mm to (70.2, 132.9)
- moved C408 0.31 mm to (80.2, 109.0)
- moved C422 0.26 mm to (80.8, 135.6)
- moved C417 0.22 mm to (82.5, 135.6)
- moved C423 0.22 mm to (86.3, 135.6)
- moved CF9 0.22 mm to (68.4, 82.3)
- moved CF15 0.22 mm to (85.8, 99.5)
- moved CF2 0.11 mm to (89.7, 96.2)
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Routing:
- net GND: track 0.00 -> 3256.7 mm, vias 0 -> 3044
- net 3V3: track 255.3 -> 260.2 mm, vias 15 -> 17
- net /STM32F4/SPI_SCK: track 22.7 -> 26.6 mm, vias 0 -> 2
- net /STM32F4/VBUS: track 131.5 -> 135.2 mm, vias 2 -> 4
- net /STM32F4/ID: track 21.8 -> 24.0 mm, vias 0 -> 2
- net /spartan6/CLK_FPGA: track 33.0 -> 31.4 mm
- net /spartan6/F_TDI: track 77.6 -> 79.0 mm
- net /STM32F4/GPIO12: track 21.8 -> 20.5 mm
- net /spartan6/IO18: track 42.8 -> 44.1 mm
- net /spartan6/IO19: track 45.4 -> 46.6 mm
- net /spartan6/IO20: track 39.1 -> 40.2 mm
- net /spartan6/F_TCK: track 121.1 -> 120.0 mm, vias 4 -> 6
- net /STM32F4/DS2: track 52.6 -> 53.7 mm
- net /STM32F4/GPIO13: track 24.0 -> 23.0 mm
- net /spartan6/IO17: track 46.4 -> 47.3 mm
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