File: SAM3S_SPARTAN6/SAM3N.sch (KiCad schematic (older format))
At the start: 28 parts, among them U11 ZLDO1117G33TA, X401 12MHz

Commit message: Routing
Parts:
- added DP3: DIODE, opendous:SM0603_Opendous, symbol DIODE
- added JMS2: USB-MINI, Connect:USB_Mini-B, symbol USB-MINI
- added RUF1, RUF2: 27, SM0603, symbol R
Connections:
- wire segments 165 -> 180
Changed lines of the file:
@@
 Text HLabel 5400 4600 2    60   Input ~ 0
 CLK_F
+$Comp
+L USB-MINI JMS2
+U 1 1 555B7046
+P 8600 3550
+F 0 "JMS2" H 8350 4000 60  0000 C CNN
+F 1 "USB-MINI" H 8500 3350 60  0000 C CNN
+F 2 "Connect:USB_Mini-B" H 8600 3550 60  0001 C CNN
+F 3 "" H 8600 3550 60  0000 C CNN
+	1    8600 3550
+	1    0    0    1
+$EndComp
+Wire Wire Line
+	7400 3550 7950 3550
+Wire Wire Line
+	7300 3650 7950 3650
+$Comp
+L GND #PWR?
+U 1 1 555B7051
+P 7750 3900
+F 0 "#PWR?" H 7750 3900 30  0001 C CNN
+F 1 "GND" H 7750 3830 30  0001 C CNN
+F 2 "" H 7750 3900 60  0001 C CNN
+F 3 "" H 7750 3900 60  0001 C CNN
+	1    7750 3900
+	1    0    0    -1
+$EndComp
+Wire Wire Line
+	7950 3850 7750 3850
+Wire Wire Line
+	7750 3850 7750 3900
+Wire Wire Line
+	9100 3500 9100 3900
+Connection ~ 9100 3700
+Connection ~ 9100 3600
+$Comp
+L DIODE DP3
+U 1 1 555B705C
+P 7800 3150
+F 0 "DP3" H 7800 3250 40  0000 C CNN
+F 1 "DIODE" H 7800 3050 40  0000 C CNN
+F 2 "opendous:SM0603_Opendous" H 7800 3150 60  0001 C CNN
+F 3 "" H 7800 3150 60  0000 C CNN
+	1    7800 3150
+	0    -1   -1   0
+$EndComp
+$Comp
+L VDD5V #PWR?
+U 1 1 555B7063
+P 7800 2850
+F 0 "#PWR?" H 7800 2950 30  0001 C CNN
+F 1 "VDD5V" H 7800 2950 30  0000 C CNN
+F 2 "" H 7800 2850 60  0001 C CNN
+F 3 "" H 7800 2850 60  0001 C CNN
+	1    7800 2850
+	1    0    0    -1
+$EndComp
+Wire Wire Line
+	7800 2850 7800 2950
+Wire Wire Line
+	7950 3450 7800 3450
+Wire Wire Line
+	7800 3450 7800 3350
+$Comp
+L GND #PWR?
+U 1 1 555B706C
+P 9100 3900
+F 0 "#PWR?" H 9100 3900 30  0001 C CNN
+F 1 "GND" H 9100 3830 30  0001 C CNN
+F 2 "" H 9100 3900 60  0001 C CNN
+F 3 "" H 9100 3900 60  0001 C CNN
+	1    9100 3900
+	1    0    0    -1
+$EndComp
+Connection ~ 9100 3800
+Wire Wire Line
+	7400 2700 7400 3550
+Wire Wire Line
+	7700 3550 7700 3550
+Wire Wire Line
+	7300 3650 7300 2800
+$Comp
+L R RUF1
+U 1 1 555B9831
+P 5950 2700
+F 0 "RUF1" V 6030 2700 50  0000 C CNN
+F 1 "27" V 5950 2700 50  0000 C CNN
+F 2 "SM0603" H 5950 2700 60  0001 C CNN
+F 3 "" H 5950 2700 60  0001 C CNN
+	1    5950 2700
+	0    1    1    0
+$EndComp
+$Comp
+L R RUF2
+U 1 1 555B9AE4
+P 6450 2800
+F 0 "RUF2" V 6530 2800 50  0000 C CNN
+F 1 "27" V 6450 2800 50  0000 C CNN
+F 2 "SM0603" H 6450 2800 60  0001 C CNN
+F 3 "" H 6450 2800 60  0001 C CNN
+	1    6450 2800
+	0    1    1    0
+$EndComp
+Wire Wire Line
+	6200 2700 7400 2700
+Wire Wire Line
+	7300 2800 6700 2800
+Wire Wire Line
+	5700 2700 4900 2700
+Wire Wire Line
+	4900 2800 6200 2800
 $EndSCHEMATC

Commit message: Finishing routing, adding gerber files
Changed lines of the file:
@@
 SAM_TX
 $Comp
-L +1.8V #PWR01
+L +1.8V #PWR05
 U 1 1 516D632A
 P 6550 8450
-F 0 "#PWR01" H 6550 8590 20  0001 C CNN
+F 0 "#PWR05" H 6550 8590 20  0001 C CNN
 F 1 "+1.8V" H 6550 8560 30  0000 C CNN
 F 2 "" H 6550 8450 60  0001 C CNN
@@
 $EndComp
 $Comp
-L GND #PWR02
+L GND #PWR06
 U 1 1 516D62F6
 P 6550 9100
-F 0 "#PWR02" H 6550 9100 30  0001 C CNN
+F 0 "#PWR06" H 6550 9100 30  0001 C CNN
 F 1 "GND" H 6550 9030 30  0001 C CNN
 F 2 "" H 6550 9100 60  0001 C CNN
@@
 $EndComp
 $Comp
-L +3.3VP #PWR03
+L +3.3VP #PWR07
 U 1 1 516D62A0
 P 6900 750
-F 0 "#PWR03" H 6950 780 20  0001 C CNN
+F 0 "#PWR07" H 6950 780 20  0001 C CNN
 F 1 "+3.3VP" H 6900 840 30  0000 C CNN
 F 2 "" H 6900 750 60  0001 C CNN
@@
 $EndComp
 $Comp
-L +3.3VP #PWR04
+L +3.3VP #PWR08
 U 1 1 516D629C
 P 7500 850
-F 0 "#PWR04" H 7550 880 20  0001 C CNN
+F 0 "#PWR08" H 7550 880 20  0001 C CNN
 F 1 "+3.3VP" H 7500 940 30  0000 C CNN
 F 2 "" H 7500 850 60  0001 C CNN
@@
 $EndComp
 $Comp
-L +3.3VP #PWR05
+L +3.3VP #PWR09
 U 1 1 516D625C
 P 4000 8450
-F 0 "#PWR05" H 4050 8480 20  0001 C CNN
+F 0 "#PWR09" H 4050 8480 20  0001 C CNN
 F 1 "+3.3VP" H 4000 8540 30  0000 C CNN
 F 2 "" H 4000 8450 60  0001 C CNN
@@
 $EndComp
 $Comp
-L +3.3VP #PWR06
+L +3.3VP #PWR010
 U 1 1 516D624A
 P 2450 800
-F 0 "#PWR06" H 2500 830 20  0001 C CNN
+F 0 "#PWR010" H 2500 830 20  0001 C CNN
 F 1 "+3.3VP" H 2450 890 30  0000 C CNN
 F 2 "" H 2450 800 60  0001 C CNN
@@
 $EndComp
 $Comp
-L GND #PWR07
+L GND #PWR011
 U 1 1 516D6095
 P 4000 9100
-F 0 "#PWR07" H 4000 9100 30  0001 C CNN
+F 0 "#PWR011" H 4000 9100 30  0001 C CNN
 F 1 "GND" H 4000 9030 30  0001 C CNN
 F 2 "" H 4000 9100 60  0001 C CNN
@@
 JTDI
 $Comp
-L GND #PWR08
+L GND #PWR012
 U 1 1 516D5EEC
 P 3250 7300
-F 0 "#PWR08" H 3250 7300 30  0001 C CNN
+F 0 "#PWR012" H 3250 7300 30  0001 C CNN
 F 1 "GND" H 3250 7230 30  0001 C CNN
 F 2 "" H 3250 7300 60  0001 C CNN
@@
 $EndComp
 $Comp
-L GND #PWR09
+L GND #PWR013
 U 1 1 516D5EBB
 P 7650 2150
-F 0 "#PWR09" H 7650 2150 30  0001 C CNN
+F 0 "#PWR013" H 7650 2150 30  0001 C CNN
 F 1 "GND" H 7650 2080 30  0001 C CNN
 F 2 "" H 7650 2150 60  0001 C CNN
@@
 $EndComp
 $Comp
-L VDD5V #PWR010
+L VDD5V #PWR014
 U 1 1 4E7B5061
 P 5450 850
-F 0 "#PWR010" H 5450 950 30  0001 C CNN
+F 0 "#PWR014" H 5450 950 30  0001 C CNN
 F 1 "VDD5V" H 5450 950 30  0000 C CNN
 F 2 "" H 5450 850 60  0001 C CNN
@@
 $EndComp
 $Comp
-L GND #PWR011
+L GND #PWR015
 U 1 1 4E7B4E89
 P 5450 1500
-F 0 "#PWR011" H 5450 1500 30  0001 C CNN
+F 0 "#PWR015" H 5450 1500 30  0001 C CNN
 F 1 "GND" H 5450 1430 30  0001 C CNN
 F 2 "" H 5450 1500 60  0001 C CNN
@@
 $EndComp
 $Comp
-L GND #PWR012
+L GND #PWR016
 U 1 1 4E7B4E84
 P 6900 1500
-F 0 "#PWR012" H 6900 1500 30  0001 C CNN
+F 0 "#PWR016" H 6900 1500 30  0001 C CNN
 F 1 "GND" H 6900 1430 30  0001 C CNN
 F 2 "" H 6900 1500 60  0001 C CNN
@@
 $EndComp
 $Comp
-L GND #PWR013
+L GND #PWR017
 U 1 1 4E7B44BE
 P 6500 1500
-F 0 "#PWR013" H 6500 1500 30  0001 C CNN
+F 0 "#PWR017" H 6500 1500 30  0001 C CNN
 F 1 "GND" H 6500 1430 30  0001 C CNN
 F 2 "" H 6500 1500 60  0001 C CNN
@@
 $EndComp
 $Comp
-L GND #PWR014
+L GND #PWR018
 U 1 1 4E7B44A2
 P 5650 1100
-F 0 "#PWR014" H 5650 1100 30  0001 C CNN
+F 0 "#PWR018" H 5650 1100 30  0001 C CNN
 F 1 "GND" H 5650 1030 30  0001 C CNN
 F 2 "" H 5650 1100 60  0001 C CNN
@@
 $EndComp
 $Comp
-L GND #PWR015
+L GND #PWR019
 U 1 1 4E188E4E
 P 9300 1350
-F 0 "#PWR015" H 9300 1350 30  0001 C CNN
+F 0 "#PWR019" H 9300 1350 30  0001 C CNN
 F 1 "GND" H 9300 1280 30  0001 C CNN
 F 2 "" H 9300 1350 60  0001 C CNN
@@
 LED
 $Comp
-L GND #PWR016
+L GND #PWR020
 U 1 1 4E186DEB
 P 8000 1350
-F 0 "#PWR016" H 8000 1350 30  0001 C CNN
+F 0 "#PWR020" H 8000 1350 30  0001 C CNN
 F 1 "GND" H 8000 1280 30  0001 C CNN
 F 2 "" H 8000 1350 60  0001 C CNN
@@
 $EndComp
 $Comp
-L +3.3VP #PWR017
+L +3.3VP #PWR021
 U 1 1 54B587C8
 P 4100 800
-F 0 "#PWR017" H 4150 830 20  0001 C CNN
+F 0 "#PWR021" H 4150 830 20  0001 C CNN
 F 1 "+3.3VP" H 4100 890 30  0000 C CNN
 F 2 "" H 4100 800 60  0001 C CNN
@@
 $EndComp
 $Comp
-L +1.8V #PWR018
+L +1.8V #PWR022
 U 1 1 516D634E
 P 3850 950
-F 0 "#PWR018" H 3850 1090 20  0001 C CNN
+F 0 "#PWR022" H 3850 1090 20  0001 C CNN
 F 1 "+1.8V" H 3850 1060 30  0000 C CNN
 F 2 "" H 3850 950 60  0001 C CNN
@@
 Wire Wire Line
 	5850 4450 6350 4450
-Text Label 6900 4450 0    60   ~ 0
-AD4
 Text Label 5900 4450 0    60   ~ 0
 AD5
@@
 LED
 $Comp
-L +3.3VP #PWR019
+L +3.3VP #PWR023
 U 1 1 54ED0F5F
-P 5850 4650
-F 0 "#PWR019" H 5900 4680 20  0001 C CNN
-F 1 "+3.3VP" H 5850 4740 30  0000 C CNN
-F 2 "" H 5850 4650 60  0001 C CNN
-F 3 "" H 5850 4650 60  0001 C CNN
-	1    5850 4650
-	0    -1   -1   0
+P 7350 4450
+F 0 "#PWR023" H 7400 4480 20  0001 C CNN
+F 1 "+3.3VP" H 7350 4540 30  0000 C CNN
+F 2 "" H 7350 4450 60  0001 C CNN
+F 3 "" H 7350 4450 60  0001 C CNN
+	1    7350 4450
+	0    1    1    0
 $EndComp
 Wire Wire Line
 	6350 4650 5850 4650
 $Comp
-L GND #PWR020
+L GND #PWR024
 U 1 1 54ED12AC
 P 7350 4650
-F 0 "#PWR020" H 7350 4650 30  0001 C CNN
+F 0 "#PWR024" H 7350 4650 30  0001 C CNN
 F 1 "GND" H 7350 4580 30  0001 C CNN
 F 2 "" H 7350 4650 60  0001 C CNN
@@
 	7300 3650 7950 3650
 $Comp
-L GND #PWR?
+L GND #PWR025
 U 1 1 555B7051
 P 7750 3900
-F 0 "#PWR?" H 7750 3900 30  0001 C CNN
+F 0 "#PWR025" H 7750 3900 30  0001 C CNN
 F 1 "GND" H 7750 3830 30  0001 C CNN
 F 2 "" H 7750 3900 60  0001 C CNN
@@
 $EndComp
 $Comp
-L VDD5V #PWR?
+L VDD5V #PWR026
 U 1 1 555B7063
 P 7800 2850
-F 0 "#PWR?" H 7800 2950 30  0001 C CNN
+F 0 "#PWR026" H 7800 2950 30  0001 C CNN
 F 1 "VDD5V" H 7800 2950 30  0000 C CNN
 F 2 "" H 7800 2850 60  0001 C CNN
@@
 	7800 3450 7800 3350
 $Comp
-L GND #PWR?
+L GND #PWR027
 U 1 1 555B706C
 P 9100 3900
-F 0 "#PWR?" H 9100 3900 30  0001 C CNN
+F 0 "#PWR027" H 9100 3900 30  0001 C CNN
 F 1 "GND" H 9100 3830 30  0001 C CNN
 F 2 "" H 9100 3900 60  0001 C CNN
@@
 Wire Wire Line
 	4900 2800 6200 2800
+$Comp
+L GND #PWR028
+U 1 1 555D26A9
+P 5850 4650
+F 0 "#PWR028" H 5850 4650 30  0001 C CNN
+F 1 "GND" H 5850 4580 30  0001 C CNN
+F 2 "" H 5850 4650 60  0001 C CNN
+F 3 "" H 5850 4650 60  0001 C CNN
+	1    5850 4650
+	0    1    1    0
+$EndComp
 $EndSCHEMATC

Commit message: Adding Examples and configuration files
Parts:
- C396, C397, C398, C399, C400, C401, C402, C403, C404, C405, C406, C407, C408, C409, C410, C411, C412, C74, C75, C76: symbol C -> C-RESCUE-i.MX283_Board
- D8, D9: symbol LED -> LED-RESCUE-i.MX283_Board
- R33, R5, RUF1, RUF2: symbol R -> R-RESCUE-i.MX283_Board
Changed lines of the file:
@@
 EESchema Schematic File Version 2
+LIBS:i.MX283_Board-rescue
 LIBS:power
 LIBS:device
@@
 LIBS:memory
 LIBS:xilinx
-LIBS:special
 LIBS:microcontrollers
 LIBS:dsp
@@
 $EndComp
 $Comp
-L C C409
+L C-RESCUE-i.MX283_Board C409
 U 1 1 516D62FA
 P 6000 8800
@@
 $EndComp
 $Comp
-L C C410
+L C-RESCUE-i.MX283_Board C410
 U 1 1 516D62F9
 P 6350 8800
@@
 $EndComp
 $Comp
-L C C411
+L C-RESCUE-i.MX283_Board C411
 U 1 1 516D62F8
 P 6700 8800
@@
 $EndComp
 $Comp
-L C C412
+L C-RESCUE-i.MX283_Board C412
 U 1 1 516D62F7
 P 7050 8800
@@
 $EndComp
 $Comp
-L GND #PWR06
+L GND-RESCUE-i.MX283_Board #PWR06
 U 1 1 516D62F6
 P 6550 9100
@@
 $EndComp
 $Comp
-L C C408
+L C-RESCUE-i.MX283_Board C408
 U 1 1 516D62F5
 P 5650 8800
@@
 $EndComp
 $Comp
-L C C401
+L C-RESCUE-i.MX283_Board C401
 U 1 1 516D60B5
 P 3100 8800
@@
 $EndComp
 $Comp
-L GND #PWR011
+L GND-RESCUE-i.MX283_Board #PWR011
 U 1 1 516D6095
 P 4000 9100
@@
 $EndComp
 $Comp
-L C C407
+L C-RESCUE-i.MX283_Board C407
 U 1 1 516D6094
 P 4500 8800
@@
 $EndComp
 $Comp
-L C C406
+L C-RESCUE-i.MX283_Board C406
 U 1 1 516D6093
 P 4150 8800
@@
 $EndComp
 $Comp
-L C C405
+L C-RESCUE-i.MX283_Board C405
 U 1 1 516D6092
 P 3800 8800
@@
 $EndComp
 $Comp
-L C C404
+L C-RESCUE-i.MX283_Board C404
 U 1 1 516D6091
 P 3450 8800
@@
 JTDI
 $Comp
-L GND #PWR012
+L GND-RESCUE-i.MX283_Board #PWR012
 U 1 1 516D5EEC
 P 3250 7300
@@
 $EndComp
 $Comp
-L GND #PWR013
+L GND-RESCUE-i.MX283_Board #PWR013
 U 1 1 516D5EBB
 P 7650 2150
@@
 $EndComp
 $Comp
-L GND #PWR015
+L GND-RESCUE-i.MX283_Board #PWR015
 U 1 1 4E7B4E89
 P 5450 1500
@@
 $EndComp
 $Comp
-L GND #PWR016
+L GND-RESCUE-i.MX283_Board #PWR016
 U 1 1 4E7B4E84
 P 6900 1500
@@
 $EndComp
 $Comp
-L C C76
+L C-RESCUE-i.MX283_Board C76
 U 1 1 4E7B4A85
 P 6900 1200
@@
 $EndComp
 $Comp
-L C C74
+L C-RESCUE-i.MX283_Board C74
 U 1 1 4E7B4A81
 P 5450 1200
@@
 $EndComp
 $Comp
-L GND #PWR017
+L GND-RESCUE-i.MX283_Board #PWR017
 U 1 1 4E7B44BE
 P 6500 1500
@@
 $EndComp
 $Comp
-L GND #PWR018
+L GND-RESCUE-i.MX283_Board #PWR018
 U 1 1 4E7B44A2
 P 5650 1100
@@
 $EndComp
 $Comp
-L C C75
+L C-RESCUE-i.MX283_Board C75
 U 1 1 4E7B41E8
 P 6500 1200
@@
 $EndComp
 $Comp
-L R R33
+L R-RESCUE-i.MX283_Board R33
 U 1 1 4E188E50
 P 8900 1350
@@
 $EndComp
 $Comp
-L LED D9
+L LED-RESCUE-i.MX283_Board D9
 U 1 1 4E188E4F
 P 8900 1050
@@
 $EndComp
 $Comp
-L GND #PWR019
+L GND-RESCUE-i.MX283_Board #PWR019
 U 1 1 4E188E4E
 P 9300 1350
@@
 LED
 $Comp
-L GND #PWR020
+L GND-RESCUE-i.MX283_Board #PWR020
 U 1 1 4E186DEB
 P 8000 1350
@@
 $EndComp
 $Comp
-L LED D8
+L LED-RESCUE-i.MX283_Board D8
 U 1 1 4DCDB178
 P 7600 1050
@@
 $EndComp
 $Comp
-L R R5
+L R-RESCUE-i.MX283_Board R5
 U 1 1 4DCDB177
 P 7600 1350
@@
 Erase
 $Comp
-L C C402
+L C-RESCUE-i.MX283_Board C402
 U 1 1 54B5643A
 P 7200 1800
@@
 $EndComp
 $Comp
-L C C403
+L C-RESCUE-i.MX283_Board C403
 U 1 1 54B5666D
 P 7200 2400
@@
 	1400 4900 1600 4900
 $Comp
-L C C398
+L C-RESCUE-i.MX283_Board C398
 U 1 1 54C403EB
 P 2100 8800
@@
 $EndComp
 $Comp
-L C C400
+L C-RESCUE-i.MX283_Board C400
 U 1 1 54C403F1
 P 2800 8800
@@
 $EndComp
 $Comp
-L C C399
+L C-RESCUE-i.MX283_Board C399
 U 1 1 54C403F7
 P 2450 8800
@@
 Connection ~ 3100 9000
 $Comp
-L C C397
+L C-RESCUE-i.MX283_Board C397
 U 1 1 54C41B07
 P 5300 8800
@@
 $EndComp
 $Comp
-L C C396
+L C-RESCUE-i.MX283_Board C396
 U 1 1 54C41B0D
 P 4950 8800
@@
 	6350 4650 5850 4650
 $Comp
-L GND #PWR024
+L GND-RESCUE-i.MX283_Board #PWR024
 U 1 1 54ED12AC
 P 7350 4650
@@
 	7300 3650 7950 3650
 $Comp
-L GND #PWR025
+L GND-RESCUE-i.MX283_Board #PWR025
 U 1 1 555B7051
 P 7750 3900
@@
 	7800 3450 7800 3350
 $Comp
-L GND #PWR027
+L GND-RESCUE-i.MX283_Board #PWR027
 U 1 1 555B706C
 P 9100 3900
@@
 	7300 3650 7300 2800
 $Comp
-L R RUF1
+L R-RESCUE-i.MX283_Board RUF1
 U 1 1 555B9831
 P 5950 2700
@@
 $EndComp
 $Comp
-L R RUF2
+L R-RESCUE-i.MX283_Board RUF2
 U 1 1 555B9AE4
 P 6450 2800
@@
 	4900 2800 6200 2800
 $Comp
-L GND #PWR028
+L GND-RESCUE-i.MX283_Board #PWR028
 U 1 1 555D26A9
 P 5850 4650

Commit message: Added files via upload
Parts:
- removed C396, C397, C398, C399, C400, C408, C409, C410: 0.1uF, SM0603, symbol C-RESCUE-i.MX283_Board
- removed C402, C403: 20pF, SM0603, symbol C-RESCUE-i.MX283_Board
- removed C411: 1uF, SM0603, symbol C-RESCUE-i.MX283_Board
- removed C412: 4.7uF, SM1206, symbol C-RESCUE-i.MX283_Board
- removed C74, C76: 33uF, SM1206, symbol C-RESCUE-i.MX283_Board
- removed C75: 100n, SM0603, symbol C-RESCUE-i.MX283_Board
- removed DP3: DIODE, opendous:SM0603_Opendous, symbol DIODE
- removed JMS2: USB-MINI, Connect:USB_Mini-B, symbol USB-MINI
- removed PSA1: CONN_02X14, Socket_Strips:Socket_Strip_Straight_2x14, symbol CONN_02X14
- removed RUF1, RUF2: 27, SM0603, symbol R-RESCUE-i.MX283_Board
- removed U11: ZLDO1117G33TA, LT1117, symbol LT1117CST
- removed US1: ATSAM3S2CA-AU, Housings_QFP:LQFP-100_14x14mm_Pitch0.5mm, symbol ATSAM3N2
- removed X401: 12MHz, ABM8G, symbol ABM8G
- added CD1: CONN_02X18, Socket_Strips:Socket_Strip_Straight_2x18, symbol CONN_02X18
- added CHB1, CHB2: 0.1uF, SM0603, symbol C-RESCUE-stamp_mini_4_layers
- added CRT1, CRT2, CS1, CS2, CST3, CST7: 0.1uF, opendous:SM0603_Opendous, symbol C-RESCUE-stamp_mini_4_layers
- added CST4: 1uF, SM0805, symbol C-RESCUE-stamp_mini_4_layers
- added CST5, CST6: 2.2uF, SMD_Packages:SMD-0603, symbol C-RESCUE-stamp_mini_4_layers
- added CXST1, CXST2: 22pF, opendous:SM0603_Opendous, symbol C-RESCUE-stamp_mini_4_layers
- added I2C1: I2C_1, Socket_Strips:Socket_Strip_Straight_2x02, symbol CONN_02X02
- added LST1, LST2: 2A 120 ohm, SM0805, symbol INDUCTOR
- added PGM1: J, Socket_Strips:Socket_Strip_Straight_1x02, symbol JUMPER
- added RST2, RST3, RST6: 10k, opendous:SM0603_Opendous, symbol R-RESCUE-stamp_mini_4_layers
- added RST4, RST5: 4.7k, opendous:SM0603_Opendous, symbol R-RESCUE-stamp_mini_4_layers
- added SW_RST1: SW_PUSH, Buttons_Switches_ThroughHole:SW_Tactile_SPST_Angled, symbol SW_PUSH
- added UST1: STM32F4_LQFP100, Housings_QFP:TQFP-100_14x14mm_Pitch0.5mm, symbol STM32F4_LQFP100
- added XRTC1: CRYSTAL, resonator:txc_32k, symbol CRYSTAL
- added XST1: 12MHz, abm8g:ABM8G, symbol ABM8G
- C401, C404, C405, C406, C407: symbol C-RESCUE-i.MX283_Board -> C-RESCUE-stamp_mini_4_layers
- D8, D9: symbol LED-RESCUE-i.MX283_Board -> LED-RESCUE-stamp_mini_4_layers
- R33, R5: symbol R-RESCUE-i.MX283_Board -> R-RESCUE-stamp_mini_4_layers
Connections:
- net labels added: 3V3, BOOT0, BOOT1, CM1A, CM1B, CM1C, CM1D, CM2A, CM2B, CM2C, CM2D, DIR_M0, DIR_M1, ECHO, FSMC_CLK, I2C1_SCL, I2C1_SDA, IO0, IO1, IO10, IO11, IO12, IO13, IO14, IO15, IO16, IO17, IO18, IO19, IO2, IO20, IO21, IO22, IO23, IO24, IO25, IO26, IO27, IO28, IO29, IO3, IO31, IO32, IO4, IO5, IO6, IO7, IO8, IO9, JTRST, NE, NOE, NRESET, NRST, NWAIT, NWE, SDIO_CK, SDIO_CMD, SDIO_D0, SDIO_D1, SDIO_D2, SDIO_D3, SP_M0, SP_M1, STM_UART_RX, STM_UART_TX, TDO, TRIGG, VDDAST, VM, VREF
- net labels removed: +1.8V, AD0, AD1, AD11, AD2, AD3, AD4, AD5, AD8, AD9, AS0, AS1, AS10, AS11, AS12, AS13, AS2, AS3, AS4, AS5, AS6, AS7, AS8, AS9, AS[0..13], CLK_F, CLK_FPGA, DS0, DS1, DS2, DS3, DS4, DS5, DS6, DS7, DS[0..7], Erase, PA1, PA2, PA27, PA28, PA29, PA3, PA30, PA4, PC10, PC14, PC16, PC9, PWMH0, PWMH1, PWMH2, PWMH3, PWML2, PWML3, RXD0, SAM_RX, SAM_TX, SNCS, SNRD, SNWAIT, SNWE, TIOA2, TXD0, URXD0, UTXD0, VDD5V
- wire segments 180 -> 207
- no-connect marks 2 -> 0
Other:
- note added: "887-1504-1-ND"
- note added: "C13"
- note added: "P10880S-ND"
- note added: "PB1\nPB0\nPC5\nPC4"
- note added: "PB8 - SCL\nPB9 - SDA"
