File: SAM3S_SPARTAN6/i.MX283_Board.sch (KiCad schematic (older format))
At the start: 0 parts

Commit message: Finishing routing, adding gerber files
Parts:
- added TH1, TH10, TH11, TH12, TH13, TH14, TH15, TH16, TH17, TH18, TH19, TH2, TH20, TH21, TH22, TH23, TH24, TH25, TH26, TH27, TH28, TH29, TH3, TH30, TH31, TH32, TH33, TH34, TH35, TH36, TH37, TH38, TH39, TH4, TH40, TH41, TH42, TH43, TH44, TH45, TH46, TH47, TH48, TH49, TH5, TH50, TH6, TH7, TH8, TH9: CONN_1, opendous:1Pin_12mil_VIA, symbol CONN_1
Connections:
- net labels added: GND
- wire segments 25 -> 30

Commit message: Added files via upload
Parts:
- removed TH1, TH10, TH11, TH12, TH13, TH14, TH15, TH16, TH17, TH18, TH19, TH2, TH20, TH21, TH22, TH23, TH24, TH25, TH26, TH27, TH28, TH29, TH3, TH30, TH31, TH32, TH33, TH34, TH35, TH36, TH37, TH38, TH39, TH4, TH40, TH41, TH42, TH43, TH44, TH45, TH46, TH47, TH48, TH49, TH5, TH50, TH6, TH7, TH8, TH9: CONN_1, opendous:1Pin_12mil_VIA, symbol CONN_1
Connections:
- net labels removed: GND
- wire segments 30 -> 29
