File: SAM3S_SPARTAN6/serial_interface.sch (KiCad schematic (older format))
At the start: 20 parts

Commit message: Adding Examples and configuration files
Parts:
- CF36, CF37, CF38, CF39, CF40, CF41: symbol C -> C-RESCUE-i.MX283_Board
- RF14, RF15, RF16, RF17, RF18, RF19, RF20, RF21: symbol R -> R-RESCUE-i.MX283_Board
Changed lines of the file:
@@
 EESchema Schematic File Version 2
+LIBS:i.MX283_Board-rescue
 LIBS:power
 LIBS:device
@@
 LIBS:memory
 LIBS:xilinx
-LIBS:special
 LIBS:microcontrollers
 LIBS:dsp
@@
 	8250 3900 9600 3900
 $Comp
-L GND #PWR059
+L GND-RESCUE-i.MX283_Board #PWR059
 U 1 1 4FC6CFCA
 P 11500 6700
@@
 $EndComp
 $Comp
-L GND #PWR060
+L GND-RESCUE-i.MX283_Board #PWR060
 U 1 1 4FC6CFB6
 P 8850 5200
@@
 $EndComp
 $Comp
-L C CF40
+L C-RESCUE-i.MX283_Board CF40
 U 1 1 4FC6CF8D
 P 9150 4800
@@
 $EndComp
 $Comp
-L C CF41
+L C-RESCUE-i.MX283_Board CF41
 U 1 1 4FC6CF5C
 P 9150 5400
@@
 $EndComp
 $Comp
-L R RF20
+L R-RESCUE-i.MX283_Board RF20
 U 1 1 4FC6C4A3
 P 13200 6100
@@
 $EndComp
 $Comp
-L +3.3V #PWR061
+L +3.3V-RESCUE-i.MX283_Board #PWR061
 U 1 1 4FC6C4A2
 P 13500 6100
+AR Path="/4FC6C4A2" Ref="#PWR061"  Part="1"
+AR Path="/555AB8C7/4FC6C4A2" Ref="#PWR061"  Part="1"
 F 0 "#PWR061" H 13500 6050 20  0001 C CNN
 F 1 "+3.3V" H 13500 6200 30  0000 C CNN
@@
 $EndComp
 $Comp
-L +3.3V #PWR062
+L +3.3V-RESCUE-i.MX283_Board #PWR062
 U 1 1 4FC6C462
 P 13500 4600
+AR Path="/4FC6C462" Ref="#PWR062"  Part="1"
+AR Path="/555AB8C7/4FC6C462" Ref="#PWR062"  Part="1"
 F 0 "#PWR062" H 13500 4550 20  0001 C CNN
 F 1 "+3.3V" H 13500 4700 30  0000 C CNN
@@
 $EndComp
 $Comp
-L R RF19
+L R-RESCUE-i.MX283_Board RF19
 U 1 1 4FC6C443
 P 13200 4600
@@
 $EndComp
 $Comp
-L GND #PWR063
+L GND-RESCUE-i.MX283_Board #PWR063
 U 1 1 4FC6C3D8
 P 10650 5750
@@
 $EndComp
 $Comp
-L C CF39
+L C-RESCUE-i.MX283_Board CF39
 U 1 1 4FC6C3C0
 P 10250 3100
@@
 $EndComp
 $Comp
-L GND #PWR064
+L GND-RESCUE-i.MX283_Board #PWR064
 U 1 1 4FC6C3BF
 P 10250 3350
@@
 $EndComp
 $Comp
-L GND #PWR067
+L GND-RESCUE-i.MX283_Board #PWR067
 U 1 1 4FC6C2CD
 P 10450 2200
@@
 $EndComp
 $Comp
-L C CF37
+L C-RESCUE-i.MX283_Board CF37
 U 1 1 4FC6C1A7
 P 10450 1950
@@
 $EndComp
 $Comp
-L GND #PWR069
+L GND-RESCUE-i.MX283_Board #PWR069
 U 1 1 4FC6C11B
 P 9650 2150
@@
 $EndComp
 $Comp
-L +3.3V #PWR070
+L +3.3V-RESCUE-i.MX283_Board #PWR070
 U 1 1 4FC6C10C
 P 12000 2800
+AR Path="/4FC6C10C" Ref="#PWR070"  Part="1"
+AR Path="/555AB8C7/4FC6C10C" Ref="#PWR070"  Part="1"
 F 0 "#PWR070" H 12000 2750 20  0001 C CNN
 F 1 "+3.3V" H 12000 2900 30  0000 C CNN
@@
 $EndComp
 $Comp
-L R RF18
+L R-RESCUE-i.MX283_Board RF18
 U 1 1 4FC6BECA
 P 11100 1950
@@
 $EndComp
 $Comp
-L C CF38
+L C-RESCUE-i.MX283_Board CF38
 U 1 1 4FC6BE12
 P 11100 2400
@@
 $EndComp
 $Comp
-L R RF16
+L R-RESCUE-i.MX283_Board RF16
 U 1 1 4FC6BD44
 P 10300 5600
@@
 $EndComp
 $Comp
-L C CF36
+L C-RESCUE-i.MX283_Board CF36
 U 1 1 4FC6BCE9
 P 9650 1900
@@
 $EndComp
 $Comp
-L GND #PWR072
+L GND-RESCUE-i.MX283_Board #PWR072
 U 1 1 4FC6BCE8
 P 11100 2650
@@
 $EndComp
 $Comp
-L +3.3V #PWR073
+L +3.3V-RESCUE-i.MX283_Board #PWR073
 U 1 1 4FC6BCE7
 P 10250 2900
+AR Path="/4FC6BCE7" Ref="#PWR073"  Part="1"
+AR Path="/555AB8C7/4FC6BCE7" Ref="#PWR073"  Part="1"
 F 0 "#PWR073" H 10250 2850 20  0001 C CNN
 F 1 "+3.3V" H 10250 3000 30  0000 C CNN
@@
 $EndComp
 $Comp
-L R RF17
+L R-RESCUE-i.MX283_Board RF17
 U 1 1 4FC6BC62
 P 10400 4500
@@
 $EndComp
 $Comp
-L R RF15
+L R-RESCUE-i.MX283_Board RF15
 U 1 1 4FC6BC59
 P 9850 4200
@@
 $EndComp
 $Comp
-L R RF14
+L R-RESCUE-i.MX283_Board RF14
 U 1 1 4FC6BC34
 P 9850 3900
@@
 	13700 4900 13700 4550
 $Comp
-L R RF21
+L R-RESCUE-i.MX283_Board RF21
 U 1 1 51CD787E
 P 13700 4300
@@
 Connection ~ 13700 4900
 $Comp
-L +3.3V #PWR075
+L +3.3V-RESCUE-i.MX283_Board #PWR075
 U 1 1 51CD7AF5
 P 13700 4000
+AR Path="/51CD7AF5" Ref="#PWR075"  Part="1"
+AR Path="/555AB8C7/51CD7AF5" Ref="#PWR075"  Part="1"
 F 0 "#PWR075" H 13700 3950 20  0001 C CNN
 F 1 "+3.3V" H 13700 4100 30  0000 C CNN
@@
 $EndComp
 $Comp
-L GND #PWR077
+L GND-RESCUE-i.MX283_Board #PWR077
 U 1 1 555AD25C
 P 7750 6000
@@
 $EndComp
 $Comp
-L GND #PWR078
+L GND-RESCUE-i.MX283_Board #PWR078
 U 1 1 555AD26D
 P 8200 4350
@@
 Connection ~ 8100 5900
 $Comp
-L GND #PWR079
+L GND-RESCUE-i.MX283_Board #PWR079
 U 1 1 555AD27C
 P 8100 6050
@@
 	8150 3900 8150 3800
 $Comp
-L GND #PWR081
+L GND-RESCUE-i.MX283_Board #PWR081
 U 1 1 555AD296
 P 6850 4350

Commit message: Added files via upload
Parts:
- CF36, CF37, CF38, CF39, CF40, CF41: symbol C-RESCUE-i.MX283_Board -> C-RESCUE-i.MX283_Board-RESCUE-i.MX283_Board
- JMS1: footprint Connect:USB_Mini-B -> CONAL:m-pad-2.1-USB-MINI-B
- PS1: footprint Connect:JACK_ALIM -> J5:J5
- RF14, RF15, RF16, RF17, RF18, RF19, RF20, RF21: symbol R-RESCUE-i.MX283_Board -> R-RESCUE-i.MX283_Board-RESCUE-i.MX283_Board
Connections:
- net labels added: VDD4P2, VDDM
- wire segments 83 -> 78
- no-connect marks 0 -> 19
