File: SAM3S_SPARTAN6/spartan6.sch (KiCad schematic (older format))
At the start: 48 parts

Commit message: Finishing routing, adding gerber files
Connections:
- net labels removed: IO1
Changed lines of the file:
@@
 $EndComp
 $Comp
-L GND #PWR021
+L GND #PWR029
 U 1 1 54C4CC43
 P 6500 9200
-F 0 "#PWR021" H 6500 9200 30  0001 C CNN
+F 0 "#PWR029" H 6500 9200 30  0001 C CNN
 F 1 "GND" H 6500 9130 30  0001 C CNN
 F 2 "" H 6500 9200 60  0001 C CNN
@@
 $EndComp
 $Comp
-L GND #PWR022
+L GND #PWR030
 U 1 1 54C4CCD4
 P 7100 5850
-F 0 "#PWR022" H 7100 5850 30  0001 C CNN
+F 0 "#PWR030" H 7100 5850 30  0001 C CNN
 F 1 "GND" H 7100 5780 30  0001 C CNN
 F 2 "" H 7100 5850 60  0001 C CNN
@@
 $EndComp
 $Comp
-L GND #PWR023
+L GND #PWR031
 U 1 1 54C4D803
 P 8800 3050
-F 0 "#PWR023" H 8800 3050 30  0001 C CNN
+F 0 "#PWR031" H 8800 3050 30  0001 C CNN
 F 1 "GND" H 8800 2980 30  0001 C CNN
 F 2 "" H 8800 3050 60  0001 C CNN
@@
 $EndComp
 $Comp
-L GND #PWR024
+L GND #PWR032
 U 1 1 54C540E0
 P 3800 8600
-F 0 "#PWR024" H 3800 8600 30  0001 C CNN
+F 0 "#PWR032" H 3800 8600 30  0001 C CNN
 F 1 "GND" H 3800 8530 30  0001 C CNN
 F 2 "" H 3800 8600 60  0001 C CNN
@@
 $EndComp
 $Comp
-L GND #PWR025
+L GND #PWR033
 U 1 1 54C569B7
 P 12250 7100
-F 0 "#PWR025" H 12250 7100 30  0001 C CNN
+F 0 "#PWR033" H 12250 7100 30  0001 C CNN
 F 1 "GND" H 12250 7030 30  0001 C CNN
 F 2 "" H 12250 7100 60  0001 C CNN
@@
 $EndComp
 $Comp
-L GND #PWR026
+L GND #PWR034
 U 1 1 54C569BD
 P 13700 7100
-F 0 "#PWR026" H 13700 7100 30  0001 C CNN
+F 0 "#PWR034" H 13700 7100 30  0001 C CNN
 F 1 "GND" H 13700 7030 30  0001 C CNN
 F 2 "" H 13700 7100 60  0001 C CNN
@@
 $EndComp
 $Comp
-L GND #PWR027
+L GND #PWR035
 U 1 1 54C569D1
 P 13300 7100
-F 0 "#PWR027" H 13300 7100 30  0001 C CNN
+F 0 "#PWR035" H 13300 7100 30  0001 C CNN
 F 1 "GND" H 13300 7030 30  0001 C CNN
 F 2 "" H 13300 7100 60  0001 C CNN
@@
 $EndComp
 $Comp
-L GND #PWR028
+L GND #PWR036
 U 1 1 54C569D7
 P 12450 6700
-F 0 "#PWR028" H 12450 6700 30  0001 C CNN
+F 0 "#PWR036" H 12450 6700 30  0001 C CNN
 F 1 "GND" H 12450 6630 30  0001 C CNN
 F 2 "" H 12450 6700 60  0001 C CNN
@@
 $EndComp
 $Comp
-L VDD5V #PWR029
+L VDD5V #PWR037
 U 1 1 54C57176
 P 10400 6400
-F 0 "#PWR029" H 10400 6500 30  0001 C CNN
+F 0 "#PWR037" H 10400 6500 30  0001 C CNN
 F 1 "VDD5V" H 10400 6500 30  0000 C CNN
 F 2 "" H 10400 6400 60  0001 C CNN
@@
 $EndComp
 $Comp
-L GND #PWR030
+L GND #PWR038
 U 1 1 54C5717C
 P 10400 7050
-F 0 "#PWR030" H 10400 7050 30  0001 C CNN
+F 0 "#PWR038" H 10400 7050 30  0001 C CNN
 F 1 "GND" H 10400 6980 30  0001 C CNN
 F 2 "" H 10400 7050 60  0001 C CNN
@@
 $EndComp
 $Comp
-L GND #PWR031
+L GND #PWR039
 U 1 1 54C57182
 P 11850 7050
-F 0 "#PWR031" H 11850 7050 30  0001 C CNN
+F 0 "#PWR039" H 11850 7050 30  0001 C CNN
 F 1 "GND" H 11850 6980 30  0001 C CNN
 F 2 "" H 11850 7050 60  0001 C CNN
@@
 $EndComp
 $Comp
-L GND #PWR032
+L GND #PWR040
 U 1 1 54C57196
 P 11450 7050
-F 0 "#PWR032" H 11450 7050 30  0001 C CNN
+F 0 "#PWR040" H 11450 7050 30  0001 C CNN
 F 1 "GND" H 11450 6980 30  0001 C CNN
 F 2 "" H 11450 7050 60  0001 C CNN
@@
 $EndComp
 $Comp
-L GND #PWR033
+L GND #PWR041
 U 1 1 54C5719C
 P 10600 6650
-F 0 "#PWR033" H 10600 6650 30  0001 C CNN
+F 0 "#PWR041" H 10600 6650 30  0001 C CNN
 F 1 "GND" H 10600 6580 30  0001 C CNN
 F 2 "" H 10600 6650 60  0001 C CNN
@@
 $EndComp
 $Comp
-L +3.3VDAC #PWR034
+L +3.3VDAC #PWR042
 U 1 1 54C574FA
 P 11850 6300
-F 0 "#PWR034" H 11850 6420 20  0001 C CNN
+F 0 "#PWR042" H 11850 6420 20  0001 C CNN
 F 1 "+3.3VDAC" H 11850 6390 30  0000 C CNN
 F 2 "" H 11850 6300 60  0000 C CNN
@@
 $EndComp
 $Comp
-L +3.3VDAC #PWR035
+L +3.3VDAC #PWR043
 U 1 1 54C576C4
 P 3800 7950
-F 0 "#PWR035" H 3800 8070 20  0001 C CNN
+F 0 "#PWR043" H 3800 8070 20  0001 C CNN
 F 1 "+3.3VDAC" H 3800 8040 30  0000 C CNN
 F 2 "" H 3800 7950 60  0000 C CNN
@@
 $EndComp
 $Comp
-L +3.3VDAC #PWR036
+L +3.3VDAC #PWR044
 U 1 1 54C578EB
 P 6850 8550
-F 0 "#PWR036" H 6850 8670 20  0001 C CNN
+F 0 "#PWR044" H 6850 8670 20  0001 C CNN
 F 1 "+3.3VDAC" H 6850 8640 30  0000 C CNN
 F 2 "" H 6850 8550 60  0000 C CNN
@@
 $EndComp
 $Comp
-L +3.3VDAC #PWR037
+L +3.3VDAC #PWR045
 U 1 1 54C57939
 P 5900 6000
-F 0 "#PWR037" H 5900 6120 20  0001 C CNN
+F 0 "#PWR045" H 5900 6120 20  0001 C CNN
 F 1 "+3.3VDAC" H 5900 6090 30  0000 C CNN
 F 2 "" H 5900 6000 60  0000 C CNN
@@
 $EndComp
 $Comp
-L +3.3VDAC #PWR038
+L +3.3VDAC #PWR046
 U 1 1 54C57C30
 P 3150 1000
-F 0 "#PWR038" H 3150 1120 20  0001 C CNN
+F 0 "#PWR046" H 3150 1120 20  0001 C CNN
 F 1 "+3.3VDAC" H 3150 1090 30  0000 C CNN
 F 2 "" H 3150 1000 60  0000 C CNN
@@
 $EndComp
 $Comp
-L +3.3VDAC #PWR039
+L +3.3VDAC #PWR047
 U 1 1 54C57F55
 P 6100 1050
-F 0 "#PWR039" H 6100 1170 20  0001 C CNN
+F 0 "#PWR047" H 6100 1170 20  0001 C CNN
 F 1 "+3.3VDAC" H 6100 1140 30  0000 C CNN
 F 2 "" H 6100 1050 60  0000 C CNN
@@
 $EndComp
 $Comp
-L +3.3VDAC #PWR040
+L +3.3VDAC #PWR048
 U 1 1 54C58093
 P 8700 1850
-F 0 "#PWR040" H 8700 1970 20  0001 C CNN
+F 0 "#PWR048" H 8700 1970 20  0001 C CNN
 F 1 "+3.3VDAC" H 8700 1940 30  0000 C CNN
 F 2 "" H 8700 1850 60  0000 C CNN
@@
 $EndComp
 $Comp
-L +3.3VDAC #PWR041
+L +3.3VDAC #PWR049
 U 1 1 54C5850A
 P 1600 4600
-F 0 "#PWR041" H 1600 4720 20  0001 C CNN
+F 0 "#PWR049" H 1600 4720 20  0001 C CNN
 F 1 "+3.3VDAC" H 1600 4690 30  0000 C CNN
 F 2 "" H 1600 4600 60  0000 C CNN
@@
 $EndComp
 $Comp
-L +1V2 #PWR042
+L +1V2 #PWR050
 U 1 1 54C59A64
 P 6750 950
-F 0 "#PWR042" H 6750 800 60  0001 C CNN
+F 0 "#PWR050" H 6750 800 60  0001 C CNN
 F 1 "+1V2" H 6750 1090 60  0000 C CNN
 F 2 "" H 6750 950 60  0000 C CNN
@@
 $EndComp
 $Comp
-L +1V2 #PWR043
+L +1V2 #PWR051
 U 1 1 54C59AD9
 P 13700 6350
-F 0 "#PWR043" H 13700 6200 60  0001 C CNN
+F 0 "#PWR051" H 13700 6200 60  0001 C CNN
 F 1 "+1V2" H 13700 6490 60  0000 C CNN
 F 2 "" H 13700 6350 60  0000 C CNN
@@
 $EndComp
 $Comp
-L +3.3VDAC #PWR044
+L +3.3VDAC #PWR052
 U 1 1 54C5AA38
 P 12250 6450
-F 0 "#PWR044" H 12250 6570 20  0001 C CNN
+F 0 "#PWR052" H 12250 6570 20  0001 C CNN
 F 1 "+3.3VDAC" H 12250 6540 30  0000 C CNN
 F 2 "" H 12250 6450 60  0000 C CNN
@@
 $EndComp
 $Comp
-L GND #PWR045
+L GND #PWR053
 U 1 1 54C5C84B
 P 6200 8600
-F 0 "#PWR045" H 6200 8600 30  0001 C CNN
+F 0 "#PWR053" H 6200 8600 30  0001 C CNN
 F 1 "GND" H 6200 8530 30  0001 C CNN
 F 2 "" H 6200 8600 60  0001 C CNN
@@
 $EndComp
 $Comp
-L +1V2 #PWR046
+L +1V2 #PWR054
 U 1 1 54C5D047
 P 6200 7950
-F 0 "#PWR046" H 6200 7800 60  0001 C CNN
+F 0 "#PWR054" H 6200 7800 60  0001 C CNN
 F 1 "+1V2" H 6200 8090 60  0000 C CNN
 F 2 "" H 6200 7950 60  0000 C CNN
@@
 SNWE
 Text Label 2850 6000 1    60   ~ 0
-IO1
+AS10
 Text Label 2950 6000 1    60   ~ 0
 IO2
@@
 IO31
 $Comp
-L +3.3VDAC #PWR047
+L +3.3VDAC #PWR055
 U 1 1 54E61B16
 P 8800 5550
-F 0 "#PWR047" H 8800 5670 20  0001 C CNN
+F 0 "#PWR055" H 8800 5670 20  0001 C CNN
 F 1 "+3.3VDAC" H 8800 5640 30  0000 C CNN
 F 2 "" H 8800 5550 60  0000 C CNN
@@
 F_TMS
 $Comp
-L GND #PWR048
+L GND #PWR056
 U 1 1 54E73BD5
 P 14250 4200
-F 0 "#PWR048" H 14250 4200 30  0001 C CNN
+F 0 "#PWR056" H 14250 4200 30  0001 C CNN
 F 1 "GND" H 14250 4130 30  0001 C CNN
 F 2 "" H 14250 4200 60  0001 C CNN
@@
 IO7
 $Comp
-L +3.3VDAC #PWR049
+L +3.3VDAC #PWR057
 U 1 1 5501F96A
 P 13000 3500
-F 0 "#PWR049" H 13000 3620 20  0001 C CNN
+F 0 "#PWR057" H 13000 3620 20  0001 C CNN
 F 1 "+3.3VDAC" H 13000 3590 30  0000 C CNN
 F 2 "" H 13000 3500 60  0000 C CNN
@@
 	12650 3500 13000 3500
 $Comp
-L GND #PWR050
+L GND #PWR058
 U 1 1 5501FF4F
 P 11750 3550
-F 0 "#PWR050" H 11750 3550 30  0001 C CNN
+F 0 "#PWR058" H 11750 3550 30  0001 C CNN
 F 1 "GND" H 11750 3480 30  0001 C CNN
 F 2 "" H 11750 3550 60  0001 C CNN

Commit message: Adding Examples and configuration files
Parts:
- CF1, CF10, CF11, CF12, CF13, CF14, CF15, CF16, CF17, CF18, CF19, CF2, CF20, CF21, CF22, CF23, CF24, CF25, CF26, CF27, CF28, CF29, CF3, CF30, CF31, CF32, CF33, CF34, CF35, CF4, CF5, CF6, CF7, CF8, CF9: symbol C -> C-RESCUE-i.MX283_Board
- DF1: symbol LED -> LED-RESCUE-i.MX283_Board
- RF1, RF2, RF3, RF4, RF5, RF6, RF7: symbol R -> R-RESCUE-i.MX283_Board
Changed lines of the file:
@@
 EESchema Schematic File Version 2
+LIBS:i.MX283_Board-rescue
 LIBS:power
 LIBS:device
@@
 LIBS:memory
 LIBS:xilinx
-LIBS:special
 LIBS:microcontrollers
 LIBS:dsp
@@
 SNWAIT
 $Comp
-L C CF11
+L C-RESCUE-i.MX283_Board CF11
 U 1 1 54C4CC3C
 P 5600 8900
@@
 $EndComp
 $Comp
-L GND #PWR029
+L GND-RESCUE-i.MX283_Board #PWR029
 U 1 1 54C4CC43
 P 6500 9200
@@
 $EndComp
 $Comp
-L C CF15
+L C-RESCUE-i.MX283_Board CF15
 U 1 1 54C4CC49
 P 7000 8900
@@
 $EndComp
 $Comp
-L C CF14
+L C-RESCUE-i.MX283_Board CF14
 U 1 1 54C4CC50
 P 6650 8900
@@
 $EndComp
 $Comp
-L C CF13
+L C-RESCUE-i.MX283_Board CF13
 U 1 1 54C4CC57
 P 6300 8900
@@
 $EndComp
 $Comp
-L C CF12
+L C-RESCUE-i.MX283_Board CF12
 U 1 1 54C4CC5E
 P 5950 8900
@@
 $EndComp
 $Comp
-L C CF8
+L C-RESCUE-i.MX283_Board CF8
 U 1 1 54C4CC71
 P 4600 8900
@@
 $EndComp
 $Comp
-L C CF10
+L C-RESCUE-i.MX283_Board CF10
 U 1 1 54C4CC78
 P 5300 8900
@@
 $EndComp
 $Comp
-L C CF9
+L C-RESCUE-i.MX283_Board CF9
 U 1 1 54C4CC7F
 P 4950 8900
@@
 $EndComp
 $Comp
-L GND #PWR030
+L GND-RESCUE-i.MX283_Board #PWR030
 U 1 1 54C4CCD4
 P 7100 5850
@@
 $EndComp
 $Comp
-L GND #PWR031
+L GND-RESCUE-i.MX283_Board #PWR031
 U 1 1 54C4D803
 P 8800 3050
@@
 Check polarity for  M0 and M1\ninit program
 $Comp
-L R RF1
+L R-RESCUE-i.MX283_Board RF1
 U 1 1 54C4EF40
 P 9050 5200
@@
 $EndComp
 $Comp
-L R RF2
+L R-RESCUE-i.MX283_Board RF2
 U 1 1 54C4F134
 P 8800 5200
@@
 $EndComp
 $Comp
-L C CF5
+L C-RESCUE-i.MX283_Board CF5
 U 1 1 54C50FB6
 P 3600 8900
@@
 $EndComp
 $Comp
-L C CF7
+L C-RESCUE-i.MX283_Board CF7
 U 1 1 54C50FBC
 P 4300 8900
@@
 $EndComp
 $Comp
-L C CF6
+L C-RESCUE-i.MX283_Board CF6
 U 1 1 54C50FC2
 P 3950 8900
@@
 $EndComp
 $Comp
-L C CF2
+L C-RESCUE-i.MX283_Board CF2
 U 1 1 54C50FCE
 P 2600 8900
@@
 $EndComp
 $Comp
-L C CF4
+L C-RESCUE-i.MX283_Board CF4
 U 1 1 54C50FD4
 P 3300 8900
@@
 $EndComp
 $Comp
-L C CF3
+L C-RESCUE-i.MX283_Board CF3
 U 1 1 54C50FDA
 P 2950 8900
@@
 $EndComp
 $Comp
-L C CF1
+L C-RESCUE-i.MX283_Board CF1
 U 1 1 54C5129A
 P 2250 8900
@@
 $EndComp
 $Comp
-L C CF18
+L C-RESCUE-i.MX283_Board CF18
 U 1 1 54C540DA
 P 2900 8300
@@
 $EndComp
 $Comp
-L GND #PWR032
+L GND-RESCUE-i.MX283_Board #PWR032
 U 1 1 54C540E0
 P 3800 8600
@@
 $EndComp
 $Comp
-L C CF22
+L C-RESCUE-i.MX283_Board CF22
 U 1 1 54C540E6
 P 4300 8300
@@
 $EndComp
 $Comp
-L C CF21
+L C-RESCUE-i.MX283_Board CF21
 U 1 1 54C540EC
 P 3950 8300
@@
 $EndComp
 $Comp
-L C CF20
+L C-RESCUE-i.MX283_Board CF20
 U 1 1 54C540F2
 P 3600 8300
@@
 $EndComp
 $Comp
-L C CF19
+L C-RESCUE-i.MX283_Board CF19
 U 1 1 54C540F8
 P 3250 8300
@@
 $EndComp
 $Comp
-L C CF17
+L C-RESCUE-i.MX283_Board CF17
 U 1 1 54C5410A
 P 2600 8300
@@
 $EndComp
 $Comp
-L C CF16
+L C-RESCUE-i.MX283_Board CF16
 U 1 1 54C543E4
 P 2250 8300
@@
 $EndComp
 $Comp
-L GND #PWR033
+L GND-RESCUE-i.MX283_Board #PWR033
 U 1 1 54C569B7
 P 12250 7100
@@
 $EndComp
 $Comp
-L GND #PWR034
+L GND-RESCUE-i.MX283_Board #PWR034
 U 1 1 54C569BD
 P 13700 7100
@@
 $EndComp
 $Comp
-L C CF32
+L C-RESCUE-i.MX283_Board CF32
 U 1 1 54C569C3
 P 13700 6800
@@
 $EndComp
 $Comp
-L C CF30
+L C-RESCUE-i.MX283_Board CF30
 U 1 1 54C569CA
 P 12250 6800
@@
 $EndComp
 $Comp
-L GND #PWR035
+L GND-RESCUE-i.MX283_Board #PWR035
 U 1 1 54C569D1
 P 13300 7100
@@
 $EndComp
 $Comp
-L GND #PWR036
+L GND-RESCUE-i.MX283_Board #PWR036
 U 1 1 54C569D7
 P 12450 6700
@@
 $EndComp
 $Comp
-L C CF31
+L C-RESCUE-i.MX283_Board CF31
 U 1 1 54C569E4
 P 13300 6800
@@
 $EndComp
 $Comp
-L GND #PWR038
+L GND-RESCUE-i.MX283_Board #PWR038
 U 1 1 54C5717C
 P 10400 7050
@@
 $EndComp
 $Comp
-L GND #PWR039
+L GND-RESCUE-i.MX283_Board #PWR039
 U 1 1 54C57182
 P 11850 7050
@@
 $EndComp
 $Comp
-L C CF34
+L C-RESCUE-i.MX283_Board CF34
 U 1 1 54C57188
 P 11850 6750
@@
 $EndComp
 $Comp
-L C CF35
+L C-RESCUE-i.MX283_Board CF35
 U 1 1 54C5718F
 P 10400 6750
@@
 $EndComp
 $Comp
-L GND #PWR040
+L GND-RESCUE-i.MX283_Board #PWR040
 U 1 1 54C57196
 P 11450 7050
@@
 $EndComp
 $Comp
-L GND #PWR041
+L GND-RESCUE-i.MX283_Board #PWR041
 U 1 1 54C5719C
 P 10600 6650
@@
 $EndComp
 $Comp
-L C CF33
+L C-RESCUE-i.MX283_Board CF33
 U 1 1 54C571A9
 P 11450 6750
@@
 $EndComp
 $Comp
-L C CF25
+L C-RESCUE-i.MX283_Board CF25
 U 1 1 54C5C845
 P 5300 8300
@@
 $EndComp
 $Comp
-L GND #PWR053
+L GND-RESCUE-i.MX283_Board #PWR053
 U 1 1 54C5C84B
 P 6200 8600
@@
 $EndComp
 $Comp
-L C CF29
+L C-RESCUE-i.MX283_Board CF29
 U 1 1 54C5C851
 P 6700 8300
@@
 $EndComp
 $Comp
-L C CF28
+L C-RESCUE-i.MX283_Board CF28
 U 1 1 54C5C857
 P 6350 8300
@@
 $EndComp
 $Comp
-L C CF27
+L C-RESCUE-i.MX283_Board CF27
 U 1 1 54C5C85D
 P 6000 8300
@@
 $EndComp
 $Comp
-L C CF26
+L C-RESCUE-i.MX283_Board CF26
 U 1 1 54C5C863
 P 5650 8300
@@
 $EndComp
 $Comp
-L C CF24
+L C-RESCUE-i.MX283_Board CF24
 U 1 1 54C5C873
 P 5000 8300
@@
 $EndComp
 $Comp
-L C CF23
+L C-RESCUE-i.MX283_Board CF23
 U 1 1 54C5C87D
 P 4650 8300
@@
 F_TMS
 $Comp
-L GND #PWR056
+L GND-RESCUE-i.MX283_Board #PWR056
 U 1 1 54E73BD5
 P 14250 4200
@@
 $EndComp
 $Comp
-L LED DF1
+L LED-RESCUE-i.MX283_Board DF1
 U 1 1 54E73BDB
 P 13850 3900
@@
 $EndComp
 $Comp
-L R RF5
+L R-RESCUE-i.MX283_Board RF5
 U 1 1 54E73BE2
 P 13850 4200
@@
 $EndComp
 $Comp
-L R RF6
+L R-RESCUE-i.MX283_Board RF6
 U 1 1 54E73D7C
 P 7850 1100
@@
 $EndComp
 $Comp
-L R RF7
+L R-RESCUE-i.MX283_Board RF7
 U 1 1 54E741C6
 P 7850 1000
@@
 $EndComp
 $Comp
-L R RF3
+L R-RESCUE-i.MX283_Board RF3
 U 1 1 54E7420C
 P 7850 900
@@
 $EndComp
 $Comp
-L R RF4
+L R-RESCUE-i.MX283_Board RF4
 U 1 1 54E7424F
 P 7850 800
@@
 	12650 3500 13000 3500
 $Comp
-L GND #PWR058
+L GND-RESCUE-i.MX283_Board #PWR058
 U 1 1 5501FF4F
 P 11750 3550

Commit message: Added files via upload
Parts:
- CF1, CF10, CF11, CF12, CF13, CF14, CF16, CF17, CF18, CF19, CF2, CF20, CF21, CF23, CF24, CF25, CF26, CF27, CF28, CF3, CF31, CF33, CF4, CF5, CF6, CF7, CF8, CF9, RF1, RF2, RF3, RF4, RF5, RF6, RF7: footprint SM0603 -> opendous:SM0603
- CF15, CF22, CF29, CF30, CF32, CF34, CF35: footprint SM1206_Opendous -> opendous:SM1206_Opendous
- DF1: footprint SM0603 -> opendous:SM0603; symbol LED-RESCUE-i.MX283_Board -> LED
- PFIO1: footprint Socket_Strips:Socket_Strip_Straight_2x18 -> CONN_18X2:pin_array_18x2
- PFIO2: footprint Socket_Strips:Socket_Strip_Straight_2x13 -> CONN_02X14:pin_array_13x2
- UF2, UF3: footprint SMD_Packages:SOT-223 -> sot:SOT223
Connections:
- net labels added: NBL0, NBL1, VDDM
- net labels removed: IO6, IO8, VDD5V
- wire segments 286 -> 350
- no-connect marks 0 -> 14
Other:
- moved on the sheet: PFIO2
